File: FlightController/FlightController.kicad_sch (KiCad schematic)
At the start: 0 parts

Commit message: wired flight computer
Parts:
- added C1, C2: 10uF, Capacitor_SMD:C_0603_1608Metric, symbol Device:C
- added C10: 1uF, Capacitor_SMD:C_0603_1608Metric, symbol Device:C
- added C11, C12: 20pF, Capacitor_SMD:C_0603_1608Metric, symbol Device:C
- added C13, C14, C15, C16, C17, C18, C19, C20, C4, C5, C6, C7, C9: 100nF, Capacitor_SMD:C_0603_1608Metric, symbol Device:C
- added C3, C8: 4.7uF, Capacitor_SMD:C_0603_1608Metric, symbol Device:C
- added D1, D2: B5819W, Diode_SMD:D_SOD-123, symbol Device:D_Schottky
- added D3: GREEN, LED_SMD:LED_0603_1608Metric, symbol Device:LED
- added D4: BLUE, LED_SMD:LED_0603_1608Metric, symbol Device:LED
- added F1: 500mA, Fuse:Fuse_1206_3216Metric, symbol Device:Polyfuse
- added J1: USB-C, Connector_USB:USB_C_Receptacle_GCT_USB4105-xx-A_16P_TopMnt_Horizontal, symbol Connector:USB_C_Receptacle_USB2.0_16P
- added J2: 5V_IN, Connector_JST:JST_GH_SM02B-GHS-TB_1x02-1MP_P1.25mm_Horizontal, symbol Connector_Generic_MountingPin:Conn_01x02_MountingPin
- added J3: SWD, Connector_JST:JST_SH_SM06B-SRSS-TB_1x06-1MP_P1.00mm_Horizontal, symbol Connector_Generic_MountingPin:Conn_01x06_MountingPin
- added J4: UART1, Connector_JST:JST_SH_SM04B-SRSS-TB_1x04-1MP_P1.00mm_Horizontal, symbol Connector_Generic_MountingPin:Conn_01x04_MountingPin
- added J5: I2C1, Connector_JST:JST_SH_SM04B-SRSS-TB_1x04-1MP_P1.00mm_Horizontal, symbol Connector_Generic_MountingPin:Conn_01x04_MountingPin
- added J6: PWM, Connector_PinHeader_2.54mm:PinHeader_1x06_P2.54mm_Vertical, symbol Connector_Generic:Conn_01x06
- added R1, R2: 5.1k, Resistor_SMD:R_0603_1608Metric, symbol Device:R
- added R10, R9: 100k, Resistor_SMD:R_0603_1608Metric, symbol Device:R
- added R11, R12, R13, R3, R8: 10k, Resistor_SMD:R_0603_1608Metric, symbol Device:R
- added R4, R5: 1k, Resistor_SMD:R_0603_1608Metric, symbol Device:R
- added R6, R7: 4.7k, Resistor_SMD:R_0603_1608Metric, symbol Device:R
- added SW1: RESET, Button_Switch_SMD:SW_SPST_TL3342, symbol Switch:SW_Push
- added SW2: BOOT, Button_Switch_SMD:SW_SPST_TL3342, symbol Switch:SW_Push
- added U1: STM32F411CEU6, FlightController:QFN-48-1EP_7x7mm_P0.5mm_EP5.6x5.6mm, symbol MCU_ST_STM32F4:STM32F411CEUx
- added U2: AP2112K-3.3, Package_TO_SOT_SMD:SOT-23-5, symbol Regulator_Linear:AP2112K-3.3
- added U3: ICM-20602, Package_LGA:LGA-16_3x3mm_P0.5mm_LayoutBorder3x5y, symbol Sensor_Motion:ICM-20602
- added U4: BMP280, Package_LGA:Bosch_LGA-8_2x2.5mm_P0.65mm_ClockwisePinNumbering, symbol Sensor_Pressure:BMP280
- added U5: W25Q128JVS, Package_SO:SOIC-8_5.3x5.3mm_P1.27mm, symbol Memory_Flash:W25Q128JVS
- added U6: USBLC6-2SC6, Package_TO_SOT_SMD:SOT-23-6, symbol Power_Protection:USBLC6-2SC6
- added Y1: 8MHz, Crystal:Crystal_SMD_3225-4Pin_3.2x2.5mm, symbol Device:Crystal_GND24
Connections:
- new net: D3.2 (A), R4.1
- new net: D4.2 (A), R5.1
- new net: D1.2 (A), F1.2
- new net +3V3: C10.1, C14.1, C15.1, C17.1, C18.1, C19.1, C2.1, C4.1, C5.1, C6.1, C7.1, C8.1, C9.1, J3.1 (Pin_1), J5.1 (Pin_1), R11.1, R12.1, R4.2, R5.2, R6.1, R7.1, R8.1, SW2.1, U1.1 (VBAT), U1.24 (VDD), U1.36 (VDD), U1.48 (VDD), U1.9 (VDDA), U2.5 (VOUT), U3.1 (VDDIO), U3.16 (VDD), U4.6 (VDDIO), U4.8 (VDD), U5.3 (~{WP}/IO_{2}), U5.7 (~{HOLD}/~{RESET}/IO_{3}), U5.8 (VCC)
- new net +5V: C1.1, D1.1 (K), D2.1 (K), J4.1 (Pin_1), J6.2 (Pin_2), R9.1, U2.1 (VIN), U2.3 (EN)
- new net BARO_CS: R12.2, U1.19 (PB1), U4.2 (CSB)
- new net BOOT0: R3.1, SW2.2, U1.44 (BOOT0)
- new net BOOT1: R13.1, U1.20 (PB2)
- new net CC1: J1.A5 (CC1), R1.1
- new net CC2: J1.B5 (CC2), R2.1
- new net FLASH_CS: R8.2, U1.25 (PB12), U5.1 (~{CS})
- new net GND: C1.2, C10.2, C11.2, C12.2, C13.2, C14.2, C15.2, C16.2, C17.2, C18.2, C19.2, C2.2, C20.2, C3.2, C4.2, C5.2, C6.2, C7.2, C8.2, C9.2, D3.1 (K), J1.A1 (GND), J1.A12 (GND), J1.B1 (GND), J1.B12 (GND), J1.SH (SHIELD), J2.2 (Pin_2), J2.MP (MountPin), J3.6 (Pin_6), J3.MP (MountPin), J4.4 (Pin_4), J4.MP (MountPin), J5.4 (Pin_4), J5.MP (MountPin), J6.1 (Pin_1), R1.2, R10.2, R13.2, R2.2, R3.2, SW1.1, U1.23 (VSS), U1.35 (VSS), U1.47 (VSS), U1.49 (VSS), U1.8 (VSSA), U2.2 (GND), U3.10 (GND), U3.11 (GND), U3.12 (GND), U3.13 (GND), U3.15 (GND), U3.8 (FSYNC), U3.9 (GND), U4.1 (GND), U4.7 (GND), U5.4 (GND), U6.2 (GND), Y1.2 (G), Y1.4 (G)
- new net I2C1_SCL: J5.2 (Pin_2), R6.2, U1.42 (PB6)
- new net I2C1_SDA: J5.3 (Pin_3), R7.2, U1.43 (PB7)
- new net IMU_CS: R11.2, U1.14 (PA4), U3.5 (~{CS})
- new net IMU_INT: U1.18 (PB0), U3.6 (INT)
- new net IMU_REGOUT: C16.1, U3.14 (REGOUT)
- new net LED_STATUS: D4.1 (K), U1.2 (PC13)
- new net NRST: C13.1, J3.4 (Pin_4), SW1.2, U1.7 (NRST)
- new net OSC_IN: C11.1, U1.5 (PH0), Y1.1
- new net OSC_OUT: C12.1, U1.6 (PH1), Y1.3
- new net PWM1: J6.3 (Pin_3), U1.40 (PB4)
- new net PWM2: J6.4 (Pin_4), U1.41 (PB5)
- new net PWM3: J6.5 (Pin_5), U1.45 (PB8)
- new net PWM4: J6.6 (Pin_6), U1.46 (PB9)
- new net SPI1_MISO: U1.16 (PA6), U3.4 (SAO/SD0), U4.5 (SDO)
- new net SPI1_MOSI: U1.17 (PA7), U3.3 (SDA/SDI), U4.3 (SDI)
- new net SPI1_SCK: U1.15 (PA5), U3.2 (SCL/SPC), U4.4 (SCK)
- new net SPI2_MISO: U1.27 (PB14), U5.2 (DO/IO_{1})
- new net SPI2_MOSI: U1.28 (PB15), U5.5 (DI/IO_{0})
- new net SPI2_SCK: U1.26 (PB13), U5.6 (CLK)
- new net SWCLK: J3.3 (Pin_3), U1.37 (PA14)
- new net SWDIO: J3.2 (Pin_2), U1.34 (PA13)
- new net SWO: J3.5 (Pin_5), U1.39 (PB3)
- new net UART1_RX: J4.3 (Pin_3), U1.31 (PA10)
- new net UART1_TX: J4.2 (Pin_2), U1.30 (PA9)
- new net USB_DM: J1.A7 (D-), J1.B7 (D-), U1.32 (PA11), U6.3 (I/O2), U6.4 (I/O2)
- new net USB_DP: J1.A6 (D+), J1.B6 (D+), U1.33 (PA12), U6.1 (I/O1), U6.6 (I/O1)
- new net VBUS: F1.1, J1.A4 (VBUS), J1.A9 (VBUS), J1.B4 (VBUS), J1.B9 (VBUS), U6.5 (VBUS)
- new net VCAP1: C3.1, U1.22 (VCAP1)
- new net VIN_EXT: D2.2 (A), J2.1 (Pin_1)
- new net VIN_SENSE: C20.1, R10.1, R9.2, U1.10 (PA0)
- no-connect marks 0 -> 10

Commit message: we chillin
Parts:
- added R14, R15: 10k, Resistor_SMD:R_0603_1608Metric, symbol Device:R
Connections:
- net +3V3: now also R14.1, R15.1; no longer U5.3 (~{WP}/IO_{2}), U5.7 (~{HOLD}/~{RESET}/IO_{3})
- net IMU_REGOUT: no longer names the net of C16.1, U3.14 (REGOUT)
- new net FLASH_HOLD: R15.2, U5.7 (~{HOLD}/~{RESET}/IO_{3})
- new net FLASH_WP: R14.2, U5.3 (~{WP}/IO_{2})
Other:
- moved on the sheet: C3, J2, R13
